File: pcb/lif-pcb/sipm-pcb.kicad_pcb (KiCad board)
At the start: 2 copper layers, 24.1 x 43.2 mm, 9 parts, among them P1 CONN_6, P2 CONN_7, U1 LM358

Commit message: Added Awesomeness. Really
Parts:
- added 1PIN: P***, 1pin, F.Cu at (19.1, -29.2)
- added 1PIN: P***, 1pin, F.Cu at (-8.89, -29.2)
- added 1PIN: P***, 1pin, F.Cu at (-8.89, 24.1)
- added 1PIN: P***, 1pin, F.Cu at (19.1, 24.1)
- C1: footprint SM0603_Capa -> C2
- R1, R2, R3: footprint SM0805 -> R3
- R4, U1: moved to F.Cu
- moved R3 289.8 mm to (20.3, -11.4), turned to 90 degrees
- moved R2 288.2 mm to (14.0, -7.62)
- moved R4 288.1 mm to (8.89, 14.0), turned to 0 degrees
- moved P2 287.0 mm to (11.4, -15.2)
- moved U1 286.0 mm to (10.2, 3.81), turned to 180 degrees
- moved P1 285.8 mm to (16.5, -12.7)
- moved R1 284.0 mm to (3.81, -10.2)
- moved C1 283.7 mm to (3.81, -2.54), turned to 90 degrees
- moved SMA_E1 260.5 mm to (29.2, -2.54), turned to 0 degrees
Connections:
- P1 pad 6: N-000003 -> N-000004
- P2 pad 3: N-000003 -> +3.3V
- P2 pad 5: GND -> N-000004
- P2 pad 7: +3.3V -> GND
Routing:
- net GND: track 0.00 -> 167.7 mm
- net +3.3V: track 0.00 -> 55.3 mm
- net N-0000010: track 0.00 -> 35.2 mm
- net N-0000011: track 0.00 -> 28.3 mm
- net N-000004: track 0.00 -> 8.89 mm
- net N-000002: track 0.00 -> 8.15 mm
- net N-000007: track 0.00 -> 6.35 mm
- net +36V: track 0.00 -> 3.81 mm
- net N-000006: track 0.00 -> 3.81 mm
- net N-000005: track 0.00 -> 3.81 mm
- net N-000001: track 0.00 -> 3.81 mm
- added copper zone on B.Cu, net GND
Other:
- board size 24.1 x 43.2 mm -> 35.6 x 61 mm
- net class Default: clearance 0.254 -> 0.5; trace_width 0.254 -> 0.5
- rule trace_clearance: 0.254 -> 0.5
