File: pcb/lif-pcb/sipm-pcb.sch (KiCad schematic (older format))
At the start: 9 parts, among them P1 CONN_6, P2 CONN_7, U1 LM358

Commit message: Added Awesomeness. Really
Connections:
- net +3.3V: now also P2.3 (P3); no longer P2.7 (P7)
- net GND: now also P2.7 (P7); no longer P2.5 (P5)
- net at P1.6: now also P2.5 (P5); no longer P2.3 (P3)
Changed lines of the file:
@@
 LIBS:valves
 LIBS:sma_edge
-LIBS:sma
 LIBS:sipm-pcb-cache
 EELAYER 27 0
@@
 Sheet 1 1
 Title "SiPM schematic"
-Date "26 mar 2014"
+Date "7 apr 2014"
 Rev ""
 Comp ""
@@
 Wire Wire Line
 	3900 2050 4700 2050
-Wire Wire Line
-	4700 2050 4700 2450
-Wire Wire Line
-	4700 2450 4950 2450
-Wire Wire Line
-	4950 2650 4900 2650
-Wire Wire Line
-	4900 2650 4900 3600
 Connection ~ 5150 3600
 Wire Wire Line
@@
 	4450 3300 4450 2950
 Wire Wire Line
-	4450 2950 4950 2950
-Wire Wire Line
-	4950 2950 4950 2850
+	4950 2450 4650 2450
+Wire Wire Line
+	4650 2450 4650 2950
+Wire Wire Line
+	4900 3600 4900 2850
+Wire Wire Line
+	4900 2850 4950 2850
+Wire Wire Line
+	4950 2650 4700 2650
+Wire Wire Line
+	4650 2950 4450 2950
+Wire Wire Line
+	4700 2650 4700 2050
 $EndSCHEMATC
